File: eagle/faros-328P-nrf8001-50x50/faros-328P-nrf8001-50x50.brd (EAGLE design)
At the start: 50 x 50 mm, 13 parts, among them IC1 ATMEGA328P-PU

Commit message: Cleaned up part names. Added BOM to readme. Added PDF showing part placement for single-sided board. Updated Gerber files and PCB layout (PDF).
Parts:
- renumbered R6 to R5, SV2 to SV1
Changed lines of the file:
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@@
 <attribute name="VALUE" x="27.2288" y="30.353" size="1.27" layer="27" ratio="10" rot="R90"/>
 </element>
-<element name="R6" library="rcl" package="0207/7" value="4.7 k" x="22.86" y="34.29" rot="R90"/>
-<element name="SV2" library="con-lstb" package="MA03-2" value="" x="41.91" y="33.02" rot="R270">
+<element name="R5" library="rcl" package="0207/7" value="4.7 k" x="22.86" y="34.29" rot="R90"/>
+<element name="SV1" library="con-lstb" package="MA03-2" value="" x="41.91" y="33.02" rot="R270">
 <attribute name="OC_NEWARK" value="unknown" x="41.91" y="33.02" size="1.778" layer="27" rot="R270" display="off"/>
 <attribute name="MPN" value="" x="41.91" y="33.02" size="1.778" layer="27" rot="R270" display="off"/>
@@
 <contactref element="C3" pad="2"/>
 <contactref element="LED1" pad="K"/>
-<contactref element="SV2" pad="6"/>
+<contactref element="SV1" pad="6"/>
 <polygon width="0.4064" layer="16">
 <vertex x="-2.54" y="50.8"/>
@@
 <signal name="N$14">
 <contactref element="IC1" pad="18"/>
-<contactref element="SV2" pad="1"/>
-<contactref element="R6" pad="1"/>
+<contactref element="SV1" pad="1"/>
+<contactref element="R5" pad="1"/>
 <wire x1="22.86" y1="30.48" x2="22.86" y2="26.67" width="0.6096" layer="16"/>
 <wire x1="22.86" y1="26.67" x2="24.13" y2="25.4" width="0.6096" layer="16"/>
@@
 <contactref element="IC1" pad="1"/>
 <contactref element="R1" pad="2"/>
-<contactref element="SV2" pad="5"/>
+<contactref element="SV1" pad="5"/>
 <wire x1="3.81" y1="7.62" x2="8.89" y2="7.62" width="0.6096" layer="16"/>
 <via x="8.89" y="10.16" extent="1-16" drill="0.8"/>
@@
 <signal name="N$2">
 <contactref element="IC1" pad="19"/>
-<contactref element="SV2" pad="3"/>
+<contactref element="SV1" pad="3"/>
 <contactref element="R3" pad="1"/>
 <wire x1="40.64" y1="33.02" x2="36.83" y2="33.02" width="0.6096" layer="16"/>
@@
 </signal>
 <signal name="N$19">
-<contactref element="SV2" pad="4"/>
+<contactref element="SV1" pad="4"/>
 <contactref element="IC1" pad="17"/>
 <contactref element="R4" pad="1"/>
@@
 <signal name="N$5">
 <contactref element="MOD1" pad="MISO"/>
-<contactref element="R6" pad="2"/>
+<contactref element="R5" pad="2"/>
 <wire x1="22.86" y1="38.1" x2="24.13" y2="39.37" width="0.6096" layer="16"/>
 <wire x1="24.13" y1="39.37" x2="30.48" y2="39.37" width="0.6096" layer="16"/>
@@
 <wire x1="26.67" y1="20.32" x2="27.94" y2="19.05" width="0.6096" layer="16"/>
 <contactref element="MOD1" pad="VDD"/>
-<contactref element="SV2" pad="2"/>
+<contactref element="SV1" pad="2"/>
 <contactref element="X1" pad="1"/>
 <contactref element="IC1" pad="20"/>
